File: Hardware/POE_Power_Supply.brd (EAGLE design)
At the start: 27.9 x 57.1 mm, 46 parts, among them J1 MAGJACK-POE, J2 USB_A_SMT_FEMALE_NS, U1 POE_PSU-DP990X, U4 3.3V

Commit message: Update x02. Fix FP for load resistor.
Parts:
- removed LOGO1, LOGO4: SFE_LOGO_NAME_FLAME.1_INCH, SparkFun-Aesthetics:SFE_LOGO_NAME_FLAME_.1
- removed U$2: (no value), output:#POE#0
- added U$19: SPARKX-LOGO4, SparkX:SPARKX-LARGE
- added U$20: (no value), output:POWER0
- added U$21: (no value), output:SUPPLY1
- added U$22: (no value), output:SUPPLY_1
- added U$7: SPARKX-LOGO4, SparkX:SPARKX-MEDIUM
- R2: value 510 -> 49.9OHM-1206-1/2W-1%; device SparkFun-Resistors:2010 -> SparkFun-Resistors:1206
- U$1: device output:ETHERNET0 -> output:#POE#0
- U$17: device output:ETHERNET0 -> output:POWER_0
- moved U$17 25.2 mm to (13.5, 22.9), flipped to the bottom, turned to 0 degrees
- moved U$1 5.54 mm to (14.0, 25.4)
- moved U$18 2.84 mm to (24.1, 44.5)
- moved U$14 0.25 mm to (14.0, 15.7)
- moved U$15 0.25 mm to (14.0, 12.2)
Routing:
- net N$9: track 6.14 -> 6.94 mm
- net GND: vias 10 -> 11
Other:
- outline, holes or cut-outs redrawn
- board text added: "x02"
- board text removed: "v10"
Changed lines of the file:
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@@
 <layer number="44" name="Drills" color="7" fill="1" visible="no" active="yes"/>
 <layer number="45" name="Holes" color="7" fill="1" visible="yes" active="yes"/>
-<layer number="46" name="Milling" color="3" fill="1" visible="no" active="yes"/>
+<layer number="46" name="Milling" color="3" fill="1" visible="yes" active="yes"/>
 <layer number="47" name="Measures" color="7" fill="1" visible="no" active="yes"/>
 <layer number="48" name="Document" color="7" fill="1" visible="no" active="yes"/>
@@
 <board>
 <plain>
-<text x="13.97" y="1.27" size="1.27" layer="16" font="vector" ratio="20" rot="SMR0" align="center">v10</text>
+<text x="13.97" y="1.27" size="1.27" layer="16" font="vector" ratio="20" rot="SMR0" align="center">x02</text>
 <text x="17.78" y="-20.32" size="1.778" layer="51" font="vector" ratio="15">N. Seidle</text>
 <wire x1="27.94" y1="0" x2="27.94" y2="57.15" width="0.05" layer="20"/>
@@
 <wire x1="0" y1="57.15" x2="0" y2="0" width="0.05" layer="20"/>
 <wire x1="27.94" y1="0" x2="0" y2="0" width="0.05" layer="20"/>
-<wire x1="11.935" y1="29.19" x2="1.968" y2="29.19" width="0.6" layer="46"/>
-<wire x1="25.905" y1="29.19" x2="15.938" y2="29.19" width="0.6" layer="46"/>
+<wire x1="11.43" y1="29.21" x2="0.762" y2="29.21" width="0.6" layer="46"/>
 <dimension x1="0" y1="0" x2="0" y2="57.15" x3="-6.35" y3="28.575" textsize="1.778" textratio="15" layer="47" unit="inch"/>
 <dimension x1="0" y1="57.15" x2="27.94" y2="57.15" x3="13.97" y3="66.04" textsize="1.778" textratio="15" layer="47" unit="inch"/>
@@
 <dimension x1="20.574" y1="-7.747" x2="20.574" y2="0" x3="31.75" y3="-3.8735" textsize="1.778" textratio="15" layer="47" unit="inch"/>
 <dimension x1="2.54" y1="2.54" x2="0" y2="2.54" x3="1.27" y3="-3.81" textsize="1.778" textratio="15" layer="47" unit="inch"/>
+<wire x1="16.51" y1="29.21" x2="26.416" y2="29.21" width="0.6" layer="46"/>
 </plain>
 <attributes>
@@
 <element name="FD3" library="SparkFun-Aesthetics" package="FIDUCIAL-MICRO" value="FIDUCIALUFIDUCIAL" x="27.305" y="0.635" smashed="yes" rot="MR270"/>
 <element name="FD4" library="SparkFun-Aesthetics" package="FIDUCIAL-MICRO" value="FIDUCIALUFIDUCIAL" x="0.635" y="56.515" smashed="yes" rot="MR270"/>
-<element name="LOGO1" library="SparkFun-Aesthetics" package="SFE_LOGO_NAME_FLAME_.1" value="SFE_LOGO_NAME_FLAME.1_INCH" x="3.81" y="45.72" smashed="yes" rot="R90"/>
 <element name="LOGO3" library="SparkFun-Aesthetics" package="OSHW-LOGO-MINI" value="OSHW-LOGOMINI" x="25.4" y="7.62" smashed="yes" rot="MR0"/>
-<element name="LOGO4" library="SparkFun-Aesthetics" package="SFE_LOGO_NAME_FLAME_.1" value="SFE_LOGO_NAME_FLAME.1_INCH" x="13.97" y="22.4" smashed="yes" rot="MR0"/>
 <element name="C3" library="SparkFun-Capacitors" package="0603" value="0.1uF" x="22.86" y="16.51" smashed="yes">
 <attribute name="NAME" x="22.86" y="17.272" size="0.6096" layer="25" font="vector" ratio="20" align="bottom-center"/>
@@
 <attribute name="VALUE" x="22.86" y="9.652" size="0.6096" layer="27" font="vector" ratio="20" rot="R180" align="top-center"/>
 </element>
-<element name="U$17" library="output" package="ETHERNET0" value="" x="24.13" y="45.72" smashed="yes" rot="R90"/>
-<element name="U$18" library="output" package="#POE#0" value="" x="26.67" y="45.72" smashed="yes" rot="R90"/>
-<element name="U$1" library="output" package="ETHERNET0" value="" x="13.97" y="19.86" smashed="yes" rot="MR0"/>
-<element name="U$2" library="output" package="#POE#0" value="" x="13.97" y="17.32" smashed="yes" rot="MR0"/>
+<element name="U$18" library="output" package="#POE#0" value="" x="24.13" y="44.45" smashed="yes" rot="R90"/>
 <element name="FRAME1" library="SparkFun-Aesthetics" package="CREATIVE_COMMONS" value="FRAME-LETTER" x="-8.89" y="-20.32" smashed="yes">
 <attribute name="DESIGNER" value="" x="-8.89" y="-20.32" size="1.778" layer="27" font="vector" ratio="15" display="off"/>
@@
 <attribute name="VALUE" x="17.907" y="13.97" size="0.6096" layer="28" font="vector" ratio="20" rot="MR90" align="top-center"/>
 </element>
-<element name="R2" library="SparkFun-Resistors" package="2010" value="510" x="13.97" y="13.97" smashed="yes">
+<element name="R2" library="SparkFun-Resistors" package="1206" value="49.9OHM-1206-1/2W-1%" x="13.97" y="13.97" smashed="yes">
 <attribute name="NAME" x="13.97" y="15.621" size="0.6096" layer="25" font="vector" ratio="20" align="bottom-center"/>
-<attribute name="PROD_ID" value="RES-08717" x="-20.32" y="-8.89" size="1.778" layer="27" font="vector" ratio="15" display="off"/>
-<attribute name="VALUE" x="13.97" y="12.319" size="0.6096" layer="27" font="vector" ratio="20" align="top-center"/>
+<attribute name="PROD_ID" value="RES-16252" x="-20.32" y="-8.89" size="1.778" layer="27" font="vector" ratio="15" display="off"/>
 </element>
 <element name="POE_LED" library="SparkFun-Jumpers" package="SMT-JUMPER_2_NC_TRACE_SILK" package3d_urn="urn:adsk.eagle:package:39281/1" value="JUMPER-SMT_2_NC_TRACE_SILK" x="6.35" y="8.89" smashed="yes" rot="MR180">
@@
 <element name="U$12" library="output" package="#GND#1" value="" x="12.7" y="7.366" smashed="yes" rot="MR270"/>
 <element name="U$13" library="output" package="#GND#1" value="" x="17.78" y="7.366" smashed="yes" rot="MR270"/>
-<element name="U$14" library="output" package="CAUTION#0" value="" x="13.97" y="16.002" smashed="yes"/>
-<element name="U$15" library="output" package="HOT1" value="" x="13.97" y="11.938" smashed="yes"/>
+<element name="U$14" library="output" package="CAUTION#0" value="" x="13.97" y="15.748" smashed="yes"/>
+<element name="U$15" library="output" package="HOT1" value="" x="13.97" y="12.192" smashed="yes"/>
 <element name="U$16" library="output" package="POE0" value="" x="3.81" y="10.287" smashed="yes"/>
+<element name="U$7" library="SparkX" package="SPARKX-MEDIUM" value="SPARKX-LOGO4" x="2.54" y="44.45" smashed="yes" rot="R90"/>
+<element name="U$19" library="SparkX" package="SPARKX-LARGE" value="SPARKX-LOGO4" x="13.97" y="33.02" smashed="yes" rot="MR0"/>
+<element name="U$20" library="output" package="POWER0" value="" x="26.67" y="40.513" smashed="yes" rot="R90"/>
+<element name="U$21" library="output" package="SUPPLY1" value="" x="26.67" y="48.26" smashed="yes" rot="R90"/>
+<element name="U$17" library="output" package="POWER_0" value="" x="13.462" y="22.86" smashed="yes" rot="MR0"/>
+<element name="U$22" library="output" package="SUPPLY_1" value="" x="13.462" y="20.32" smashed="yes" rot="MR0"/>
+<element name="U$1" library="output" package="#POE#0" value="" x="13.97" y="25.4" smashed="yes" rot="MR0"/>
 </elements>
 <signals>
@@
 <via x="6.35" y="6.35" extent="1-16" drill="0.381"/>
 <via x="10.16" y="15.748" extent="1-16" drill="0.381"/>
-<via x="13.97" y="15.24" extent="1-16" drill="0.381"/>
-<via x="19.05" y="20.066" extent="1-16" drill="0.381"/>
+<via x="10.795" y="13.462" extent="1-16" drill="0.381"/>
+<via x="19.304" y="18.034" extent="1-16" drill="0.381"/>
 <via x="25.4" y="16.51" extent="1-16" drill="0.381"/>
 <via x="25.4" y="19.05" extent="1-16" drill="0.381"/>
 <via x="20.32" y="8.89" extent="1-16" drill="0.381"/>
 <via x="17.399" y="4.191" extent="1-16" drill="0.381"/>
-<wire x1="23.71" y1="19.05" x2="25.4" y2="19.05" width="0" layer="19" extent="1-1"/>
-<wire x1="25.4" y1="16.51" x2="25.4" y2="19.05" width="0" layer="19" extent="1-1"/>
-<wire x1="23.71" y1="16.51" x2="25.4" y2="16.51" width="0" layer="19" extent="1-1"/>
-<wire x1="22.86" y1="14.0001" x2="23.71" y2="16.51" width="0" layer="19" extent="1-1"/>
-<wire x1="22.86" y1="12.7" x2="22.86" y2="14.0001" width="0" layer="19" extent="1-1"/>
-<wire x1="22.01" y1="8.89" x2="22.86" y2="12.7" width="0" layer="19" extent="1-1"/>
-<wire x1="20.32" y1="8.89" x2="22.01" y2="8.89" width="0" layer="19" extent="1-1"/>
-<wire x1="17.78" y1="10.16" x2="20.32" y2="8.89" width="0" layer="19" extent="1-1"/>
-<wire x1="17.399" y1="4.191" x2="17.47" y2="6.752" width="0" layer="19" extent="1-1"/>
-<wire x1="20.76" y1="22.11" x2="23.71" y2="19.05" width="0" layer="19" extent="1-1"/>
-<wire x1="19.05" y1="20.066" x2="20.76" y2="22.11" width="0" layer="19" extent="1-1"/>
-<wire x1="17.78" y1="18.68" x2="19.05" y2="20.066" width="0" layer="19" extent="1-1"/>
-<wire x1="12.7" y1="10.16" x2="17.78" y2="10.16" width="0" layer="19" extent="1-1"/>
-<wire x1="11.77" y1="13.97" x2="12.7" y2="10.16" width="0" layer="19" extent="1-1"/>
-<wire x1="10.16" y1="15.748" x2="11.77" y2="13.97" width="0" layer="19" extent="1-1"/>
-<wire x1="10.16" y1="16.88" x2="10.16" y2="15.748" width="0" layer="19" extent="1-1"/>
-<wire x1="12.7" y1="16.88" x2="10.16" y2="16.88" width="0" layer="19" extent="1-1"/>
-<wire x1="13.97" y1="15.24" x2="12.7" y2="16.88" width="0" layer="19" extent="1-1"/>
-<wire x1="5.08" y1="15.24" x2="10.16" y2="15.748" width="0" layer="19" extent="1-1"/>
-<wire x1="5.08" y1="12.84" x2="5.08" y2="15.24" width="0" layer="19" extent="1-1"/>
-<wire x1="4.687" y1="8.89" x2="5.08" y2="12.84" width="0" layer="19" extent="1-1"/>
-<wire x1="6.35" y1="6.35" x2="4.687" y2="8.89" width="0" layer="19" extent="1-1"/>
-<wire x1="2.54" y1="24.13" x2="5.08" y2="15.24" width="0" layer="19" extent="1-1"/>
+<via x="20.701" y="25.019" extent="1-16" drill="0.381"/>
 </signal>
 <signal name="3.3V">
@@
 <wire x1="20.574" y1="13.462" x2="19.05" y2="13.462" width="0.5588" layer="1"/>
 <wire x1="19.05" y1="13.462" x2="18.542" y2="13.97" width="0.5588" layer="1"/>
-<wire x1="18.542" y1="13.97" x2="16.17" y2="13.97" width="0.5588" layer="1"/>
+<wire x1="18.542" y1="13.97" x2="15.37" y2="13.97" width="0.5588" layer="1"/>
 </signal>
 <signal name="N$6">
