File: Hardware/POE_Power_Supply.sch (EAGLE design)
At the start: 28 parts, among them J1 MAGJACK_SYM, J2 USB_A_SMT_FEMALE_NS, U1 POE_PSU-DP990X, U4 3.3V

Commit message: Add silk labels. Remove backup files. Add ignore.
Parts:
- J1: value MAGJACK_SYM -> MAGJACK-POE; device Ethernet:MAGJACK_SYM -> SparkFun-Connectors:MAGJACK-POE
- U1: device Ethernet:POE_PSU-DP990X -> SparkFun-IC-Power:POE_PSU-DP990X
Other:
- note added: "20mV at 40kHz"
- note added: "VPP 20mV at 200kHz"
- note added: "~93ma"

Commit message: Update x02. Fix FP for load resistor.
Parts:
- removed LOGO1: SFE_LOGO_NAME_FLAME.1_INCH, SparkFun-Aesthetics:SFE_LOGO_NAME_FLAME.1_INCH
- added U$7: SPARKX-LOGO4, SparkX:SPARKX-LOGO4
- R2: value 510 -> 49.9OHM-1206-1/2W-1%; device SparkFun-Resistors:510OHM-2010-1/2W-5% -> SparkFun-Resistors:49.9OHM-1206-1/2W-1%
Changed lines of the file:
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@@
 <part name="FD3" library="SparkFun-Aesthetics" deviceset="FIDUCIAL" device="UFIDUCIAL"/>
 <part name="FD4" library="SparkFun-Aesthetics" deviceset="FIDUCIAL" device="UFIDUCIAL"/>
-<part name="LOGO1" library="SparkFun-Aesthetics" deviceset="SFE_LOGO_NAME_FLAME" device=".1_INCH"/>
 <part name="LOGO3" library="SparkFun-Aesthetics" deviceset="OSHW-LOGO" device="MINI"/>
 <part name="SUPPLY3" library="SparkFun-PowerSymbols" deviceset="5V" device=""/>
@@
 <part name="LOAD" library="SparkFun-Jumpers" deviceset="JUMPER-SMT_2_NC_TRACE" device="_SILK" package3d_urn="urn:adsk.eagle:package:39281/1" value="JUMPER-SMT_2_NC_TRACE_SILK"/>
 <part name="GND31" library="SparkFun-PowerSymbols" deviceset="GND" device=""/>
-<part name="R2" library="SparkFun-Resistors" deviceset="510OHM" device="-2010-1/2W-5%" value="510"/>
+<part name="R2" library="SparkFun-Resistors" deviceset="49.9OHM" device="-1206-1/2W-1%" value="49.9OHM-1206-1/2W-1%"/>
 <part name="POE_LED" library="SparkFun-Jumpers" deviceset="JUMPER-SMT_2_NC_TRACE" device="_SILK" package3d_urn="urn:adsk.eagle:package:39281/1" value="JUMPER-SMT_2_NC_TRACE_SILK"/>
 <part name="R11" library="SparkFun-Resistors" deviceset="1KOHM" device="-0603-1/10W-1%" value="1k"/>
 <part name="D5" library="SparkFun-LED" deviceset="LED-RED" device="0603" value="RED"/>
 <part name="GND27" library="SparkFun-PowerSymbols" deviceset="GND" device=""/>
+<part name="U$7" library="SparkX" deviceset="SPARKX-LOGO" device="4"/>
 </parts>
 <sheets>
@@
 <instance part="FD3" gate="G$1" x="246.38" y="25.4" smashed="yes"/>
 <instance part="FD4" gate="G$1" x="243.84" y="25.4" smashed="yes"/>
-<instance part="LOGO1" gate="G$1" x="147.32" y="35.56" smashed="yes"/>
 <instance part="LOGO3" gate="G$1" x="236.22" y="45.72" smashed="yes"/>
 <instance part="SUPPLY3" gate="G$1" x="185.42" y="154.94" smashed="yes">
@@
 <attribute name="VALUE" x="137.16" y="121.666" size="1.778" layer="96" align="top-center"/>
 </instance>
-<instance part="R2" gate="G$1" x="137.16" y="132.08" smashed="yes" rot="R90">
+<instance part="R2" gate="R1" x="137.16" y="132.08" smashed="yes" rot="R90">
 <attribute name="NAME" x="135.636" y="132.08" size="1.778" layer="95" font="vector" rot="R90" align="bottom-center"/>
-<attribute name="VALUE" x="138.684" y="132.08" size="1.778" layer="96" font="vector" rot="R90" align="top-center"/>
 </instance>
 <instance part="POE_LED" gate="G$1" x="147.32" y="144.78" smashed="yes" rot="R90">
@@
 <attribute name="VALUE" x="147.32" y="111.506" size="1.778" layer="96" align="top-center"/>
 </instance>
+<instance part="U$7" gate="G$1" x="208.28" y="45.72" smashed="yes"/>
 </instances>
 <busses>
@@
 <pinref part="GND31" gate="1" pin="GND"/>
 <wire x1="137.16" y1="124.46" x2="137.16" y2="127" width="0.1524" layer="91"/>
-<pinref part="R2" gate="G$1" pin="1"/>
+<pinref part="R2" gate="R1" pin="1"/>
 </segment>
 <segment>
@@
 <pinref part="LOAD" gate="G$1" pin="1"/>
 <wire x1="137.16" y1="137.16" x2="137.16" y2="139.7" width="0.1524" layer="91"/>
-<pinref part="R2" gate="G$1" pin="2"/>
-</segment>
-</net>
+<pinref part="R2" gate="R1" pin="2"/>
+</segment>
+</net>

Commit message: Add schematic
Other:
- note removed: "20mV at 40kHz"
- note removed: "Add PTC?"
- note removed: "VPP 20mV at 200kHz"
- note removed: "~93ma"
Changed lines of the file:
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@@
 <text x="117.094" y="167.386" size="2.54" layer="94" font="vector" align="center">Power Over Ethernet</text>
 <text x="129.54" y="114.3" size="1.778" layer="97" font="vector" align="center">Dummy Load: 100mA</text>
-<text x="7.62" y="193.04" size="1.27" layer="91">Add PTC?</text>
-<text x="7.62" y="190.5" size="1.27" layer="91">~93ma</text>
-<text x="7.62" y="187.96" size="1.27" layer="91">VPP 20mV at 200kHz</text>
-<text x="7.62" y="185.42" size="1.27" layer="91">20mV at 40kHz</text>
 </plain>
 <instances>
@@
 <instance part="LOAD" gate="G$1" x="137.16" y="144.78" smashed="yes" rot="R90">
 <attribute name="NAME" x="135.128" y="142.24" size="1.778" layer="95" font="vector" rot="R90"/>
-<attribute name="VALUE" x="139.7" y="134.62" size="1.778" layer="96" font="vector" rot="R90" align="top-left"/>
 </instance>
 <instance part="GND31" gate="1" x="137.16" y="121.92" smashed="yes">
@@
 <instance part="POE_LED" gate="G$1" x="147.32" y="144.78" smashed="yes" rot="R90">
 <attribute name="NAME" x="145.288" y="139.954" size="1.778" layer="95" font="vector" rot="R90"/>
-<attribute name="VALUE" x="149.86" y="134.62" size="1.778" layer="96" font="vector" rot="R90" align="top-left"/>
 </instance>
 <instance part="R11" gate="G$1" x="147.32" y="132.08" smashed="yes" rot="R90">
